File: Praxis_BeeFreq/Praxis_BeeFreq.kicad_pcb (KiCad board)
At the start: 2 copper layers, 39.5 x 16 mm, 23 parts, among them J1 Conn_01x03_Pin, U1 NE5532DR, U2 NE5532DR

Commit message: Changes
Parts:
- moved C2 0.33 mm to (42.4, 44.2)
- moved R12 0.26 mm to (54.0, 46.7)
Routing:
- net Net-(U1-2IN-): track 22.7 -> 21.8 mm
- net Net-(U1-2IN+): track 14.1 -> 13.5 mm
Other:
- board size 39.5 x 16 mm -> 46.4 x 16 mm
Changed lines of the file:
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@@
 	(footprint "Resistor_SMD:R_0805_2012Metric"
 		(layer "F.Cu")
-		(at 54 47 180)
+		(at 54 46.736 180)
 		(descr "Resistor SMD 0805 (2012 Metric), square (rectangular) end terminal, IPC_7351 nominal, (Body size source: IPC-SM-782 page 72, https://www.pcb-3d.com/wordpress/wp-content/uploads/ipc-sm-782a_amendment_1_and_2.pdf), generated with kicad-footprint-generator")
 		(tags "resistor")
@@
 	(footprint "Capacitor_SMD:C_0805_2012Metric"
 		(layer "F.Cu")
-		(at 42.55 44.5)
+		(at 42.418 44.196)
 		(descr "Capacitor SMD 0805 (2012 Metric), square (rectangular) end terminal, IPC_7351 nominal, (Body size source: IPC-SM-782 page 76, https://www.pcb-3d.com/wordpress/wp-content/uploads/ipc-sm-782a_amendment_1_and_2.pdf, https://docs.google.com/spreadsheets/d/1BsfQQcO9C6DZCsRaXUlFlo91Tg2WpOkGARC1WS5S8t0/edit?usp=sharing), generated with kicad-footprint-generator")
 		(tags "capacitor")
@@
 	)
 	(gr_rect
-		(start 35.5 32.5)
+		(start 28.642 32.5)
 		(end 75 48.5)
 		(stroke
@@
 	(gr_text "Team 50 - Design 1"
 		(at 58 35 0)
-		(layer "F.SilkS")
+		(layer "F.SilkS" knockout)
 		(effects
 			(font
 				(size 1 1)
-				(thickness 0.1)
+				(thickness 0.2)
+				(bold yes)
 			)
 			(justify left bottom)
@@
 	)
 	(segment
-		(start 43.4125 44.4125)
-		(end 43.5 44.5)
+		(start 43.4125 42)
+		(end 43.5 42.0875)
 		(width 0.2)
 		(layer "F.Cu")
@@
 	)
 	(segment
-		(start 43.4125 42)
-		(end 43.4125 44.4125)
+		(start 43.5 42.0875)
+		(end 43.5 44.5)
 		(width 0.2)
 		(layer "F.Cu")
@@
 	)
 	(segment
-		(start 37 42)
-		(end 39.1 42)
+		(start 41.6 44.196)
+		(end 41.6 46.9875)
 		(width 0.2)
 		(layer "F.Cu")
@@
 	)
 	(segment
-		(start 41.6 44.5)
-		(end 41.6 46.9875)
+		(start 41.6 46.9875)
+		(end 41.5875 47)
 		(width 0.2)
 		(layer "F.Cu")
@@
 	)
 	(segment
-		(start 41.6 46.9875)
-		(end 41.5875 47)
+		(start 37 42)
+		(end 39.404 42)
 		(width 0.2)
 		(layer "F.Cu")
@@
 	)
 	(segment
-		(start 39.1 42)
-		(end 41.6 44.5)
+		(start 39.404 42)
+		(end 41.6 44.196)
 		(width 0.2)
 		(layer "F.Cu")
@@
 	)
 	(segment
-		(start 54.9 40.1)
-		(end 54.9 39.5)
+		(start 54.102 45.9255)
+		(end 54.9125 46.736)
 		(width 0.2)
 		(layer "F.Cu")
@@
 	)
 	(segment
-		(start 53.851 42.851)
-		(end 53.851 45.9385)
+		(start 53 42)
+		(end 53 42.725)
 		(width 0.2)
 		(layer "F.Cu")
@@
 	)
 	(segment
-		(start 53.851 45.9385)
-		(end 54.9125 47)
+		(start 53 42.725)
+		(end 54.102 43.827)
 		(width 0.2)
 		(layer "F.Cu")
@@
 	)
 	(segment
-		(start 53 42)
-		(end 53.851 42.851)
+		(start 54.9 40.1)
+		(end 54.9 39.5)
 		(width 0.2)
 		(layer "F.Cu")
@@
 	)
 	(segment
-		(start 57.9 39)
-		(end 54.9 42)
+		(start 54.102 43.827)
+		(end 54.102 45.9255)
 		(width 0.2)
 		(layer "F.Cu")
-		(net 11)
+		(net 10)
 	)
 	(segment
-		(start 48.850001 45)
-		(end 52 45)
+		(start 57.9 39)
+		(end 54.9 42)
 		(width 0.2)
 		(layer "F.Cu")
@@
 	)
 	(segment
-		(start 54.49335 43.301554)
-		(end 54.49335 42.40665)
+		(start 49.022 44.704)
+		(end 48.850001 44.875999)
 		(width 0.2)
 		(layer "F.Cu")
@@
 	)
 	(segment
-		(start 48.365 45.485001)
-		(end 48.850001 45)
+		(start 48.850001 45)
+		(end 48.365 45.485001)
 		(width 0.2)
 		(layer "F.Cu")
@@
 	)
 	(segment
-		(start 54.49335 42.40665)
-		(end 54.9 42)
+		(start 48.850001 44.875999)
+		(end 48.850001 45)
 		(width 0.2)
 		(layer "F.Cu")
@@
 	)
 	(segment
-		(start 48.365 46.47)
-		(end 48.365 45.485001)
+		(start 48.365 45.485001)
+		(end 48.365 46.47)
 		(width 0.2)
 		(layer "F.Cu")
@@
 	)
 	(via
-		(at 54.49335 43.301554)
+		(at 54.9 42)
 		(size 0.6)
 		(drill 0.3)
@@
 	)
 	(via
-		(at 52 45)
+		(at 49.022 44.704)
 		(size 0.6)
 		(drill 0.3)
@@
 	)
 	(segment
-		(start 52 44.700057)
-		(end 53.398503 43.301554)
+		(start 50.201729 44.704)
+		(end 49.022 44.704)
+		(width 0.2)
+		(layer "B.Cu")
+		(net 11)
+	)
+	(segment
+		(start 53.266057 43.434)
+		(end 51.471729 43.434)
 		(width 0.2)
 		(layer "B.Cu")
@@
 	(segment
 		(start 53.398503 43.301554)
-		(end 54.49335 43.301554)
+		(end 53.266057 43.434)
+		(width 0.2)
+		(layer "B.Cu")
+		(net 11)
+	)
+	(segment
+		(start 51.471729 43.434)
+		(end 50.201729 44.704)
 		(width 0.2)
 		(layer "B.Cu")
@@
 	)
 	(segment
-		(start 52 45)
-		(end 52 44.700057)
+		(start 53.598446 43.301554)
+		(end 53.398503 43.301554)
+		(width 0.2)
+		(layer "B.Cu")
+		(net 11)
+	)
+	(segment
+		(start 54.9 42)
+		(end 53.598446 43.301554)
 		(width 0.2)
 		(layer "B.Cu")
@@
 	)
 	(segment
-		(start 50.079001 47.899)
-		(end 52.1885 47.899)
-		(width 0.2)
-		(layer "F.Cu")
-		(net 15)
-	)
-	(segment
-		(start 66.225 47)
-		(end 65 47)
+		(start 49.635 46.47)
+		(end 49.635 46.868824)
 		(width 0.2)
 		(layer "F.Cu")
@@
 	)
 	(segment
-		(start 47.095 46.47)
-		(end 47.095 46.868824)
+		(start 49.635 46.868824)
+		(end 50.522176 47.756)
 		(width 0.2)
 		(layer "F.Cu")
@@
 	)
 	(segment
-		(start 49.635 47.454999)
-		(end 50.079001 47.899)
+		(start 66.225 47)
+		(end 65 47)
 		(width 0.2)
 		(layer "F.Cu")
@@
 	)
 	(segment
-		(start 49.635 46.868824)
-		(end 49.635 46.47)
+		(start 47.095 46.47)
+		(end 47.095 46.868824)
 		(width 0.2)
 		(layer "F.Cu")
@@
 	)
 	(segment
-		(start 52.1885 47.899)
+		(start 52.3315 47.756)
 		(end 53.0875 47)
 		(width 0.2)
@@
 	)
 	(segment
-		(start 49.635 46.47)
-		(end 49.635 47.454999)
+		(start 47.095 46.868824)
+		(end 47.982176 47.756)
 		(width 0.2)
 		(layer "F.Cu")
@@
 	)
 	(segment
-		(start 47.095 46.868824)
-		(end 47.982176 47.756)
+		(start 47.982176 47.756)
+		(end 48.747824 47.756)
 		(width 0.2)
 		(layer "F.Cu")
@@
 	)
 	(segment
-		(start 47.982176 47.756)
-		(end 48.747824 47.756)
+		(start 50.522176 47.756)
+		(end 52.3315 47.756)
 		(width 0.2)
 		(layer "F.Cu")
@@
 		(hatch edge 0.5)
 		(connect_pads
-			(clearance 0.5)
+			(clearance 0.15)
 		)
 		(min_thickness 0.25)
 		(filled_areas_thickness no)
-		(fill
+		(fill yes
 			(thermal_gap 0.5)
 			(thermal_bridge_width 0.5)
@@
 		(priority 1)
 		(connect_pads
-			(clearance 0.5)
+			(clearance 0.15)
 		)
 		(min_thickness 0.25)
 		(filled_areas_thickness no)
-		(fill
+		(fill yes
 			(thermal_gap 0.5)
 			(thermal_bridge_width 0.5)

Commit message: BetterVersion
Parts:
- MK2: footprint Connector_Wire:SolderWire-0.1sqmm_1x02_P3.6mm_D0.4mm_OD1mm -> Connector_Wire:SolderWire-2sqmm_1x02_P7.8mm_D2mm_OD3.9mm
- moved C1 6.50 mm to (58.0, 36.0)
- moved R1 6.50 mm to (60.5, 36.0)
- moved R3 6.50 mm to (55.5, 36.0)
- moved MK2 1.00 mm to (43.2, 35.5)
Connections:
- MK2 pad 1: (no net) -> GND
- MK2 pad 2: (no net) -> Net-(C1-Pad1)
Routing:
- net Net-(C1-Pad1): track 2.52 -> 10.1 mm
- net Net-(U1-1IN-): track 4.84 -> 10.1 mm
- net GND: vias 9 -> 7
Other:
- board text added: "Team 50 Design 1"
- board text removed: "Team 50 - Design 1"
Changed lines of the file:
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@@
 	)
 	(setup
+		(stackup
+			(layer "F.SilkS"
+				(type "Top Silk Screen")
+			)
+			(layer "F.Paste"
+				(type "Top Solder Paste")
+			)
+			(layer "F.Mask"
+				(type "Top Solder Mask")
+				(thickness 0.01)
+			)
+			(layer "F.Cu"
+				(type "copper")
+				(thickness 0.035)
+			)
+			(layer "dielectric 1"
+				(type "core")
+				(thickness 1.51)
+				(material "FR4")
+				(epsilon_r 4.5)
+				(loss_tangent 0.02)
+			)
+			(layer "B.Cu"
+				(type "copper")
+				(thickness 0.035)
+			)
+			(layer "B.Mask"
+				(type "Bottom Solder Mask")
+				(thickness 0.01)
+			)
+			(layer "B.Paste"
+				(type "Bottom Solder Paste")
+			)
+			(layer "B.SilkS"
+				(type "Bottom Silk Screen")
+			)
+			(copper_finish "None")
+			(dielectric_constraints no)
+		)
 		(pad_to_mask_clearance 0)
 		(allow_soldermask_bridges_in_footprints no)
@@
 	(footprint "Capacitor_SMD:C_0805_2012Metric"
 		(layer "F.Cu")
-		(at 51.5 35.95 90)
+		(at 58 35.95 90)
 		(descr "Capacitor SMD 0805 (2012 Metric), square (rectangular) end terminal, IPC_7351 nominal, (Body size source: IPC-SM-782 page 76, https://www.pcb-3d.com/wordpress/wp-content/uploads/ipc-sm-782a_amendment_1_and_2.pdf, https://docs.google.com/spreadsheets/d/1BsfQQcO9C6DZCsRaXUlFlo91Tg2WpOkGARC1WS5S8t0/edit?usp=sharing), generated with kicad-footprint-generator")
 		(tags "capacitor")
@@
 	(footprint "Resistor_SMD:R_0805_2012Metric"
 		(layer "F.Cu")
-		(at 54 35.95 -90)
+		(at 60.5 35.95 -90)
 		(descr "Resistor SMD 0805 (2012 Metric), square (rectangular) end terminal, IPC_7351 nominal, (Body size source: IPC-SM-782 page 72, https://www.pcb-3d.com/wordpress/wp-content/uploads/ipc-sm-782a_amendment_1_and_2.pdf), generated with kicad-footprint-generator")
 		(tags "resistor")
@@
 		)
 		(embedded_fonts no)
+		(model "/Users/annagavrileva/Desktop/CMA-4544PF-W--3DModel-STEP-1.STEP"
+			(offset
+				(xyz 0 0 0)
+			)
+			(scale
+				(xyz 1 1 1)
+			)
+			(rotate
+				(xyz -90 -0 180)
+			)
+		)
 	)
 	(footprint "Capacitor_SMD:C_0805_2012Metric"
@@
 		)
 		(embedded_fonts no)
+		(model "/Users/annagavrileva/Desktop/NE5532DR.STEP"
+			(offset
+				(xyz 0 0 0)
+			)
+			(scale
+				(xyz 1 1 1)
+			)
+			(rotate
+				(xyz -90 -0 -0)
+			)
+		)
 	)
 	(footprint "Resistor_SMD:R_0805_2012Metric"
@@
 		)
 	)
-	(footprint "Connector_Wire:SolderWire-0.1sqmm_1x02_P3.6mm_D0.4mm_OD1mm"
+	(footprint "Connector_Wire:SolderWire-2sqmm_1x02_P7.8mm_D2mm_OD3.9mm"
 		(layer "F.Cu")
-		(at 42.2 35.5)
-		(descr "Soldered wire connection, for 2 times 0.1 mm² wires, basic insulation, conductor diameter 0.4mm, outer diameter 1mm, size source Multi-Contact FLEXI-E 0.1 (https://ec.staubli.com/AcroFiles/Catalogues/TM_Cab-Main-11014119_(en)_hi.pdf), bend radius 3 times outer diameter, generated with kicad-footprint-generator")
-		(tags "connector wire 0.1sqmm")
+		(at 43.2 35.5)
+		(descr "Soldered wire connection, for 2 times 2 mm² wires, reinforced insulation, conductor diameter 2mm, outer diameter 3.9mm, size source Multi-Contact FLEXI-xV 2.0 (https://ec.staubli.com/AcroFiles/Catalogues/TM_Cab-Main-11014119_(en)_hi.pdf), bend radius 3 times outer diameter, generated with kicad-footprint-generator")
+		(tags "connector wire 2sqmm")
 		(property "Reference" "MK2"
-			(at 1.8 -2 0)
+			(at -4.7 -1.5 0)
 			(layer "F.SilkS")
 			(effects
@@
 		)
 		(property "Value" "CMA-6542PF"
-			(at 1.8 2 0)
+			(at 2.9 4 0)
 			(layer "F.Fab")
 			(hide yes)
@@
 		(attr exclude_from_pos_files)
 		(fp_line
-			(start -1.3 -1.3)
-			(end -1.3 1.3)
+			(start -2.7 -2.45)
+			(end -2.7 2.45)
 			(stroke
 				(width 0.05)
@@
 		)
 		(fp_line
-			(start -1.3 1.3)
-			(end 1.3 1.3)
+			(start -2.7 2.45)
+			(end 2.7 2.45)
 			(stroke
 				(width 0.05)
@@
 		)
 		(fp_line
-			(start 1.3 -1.3)
-			(end -1.3 -1.3)
+			(start 2.7 -2.45)
+			(end -2.7 -2.45)
 			(stroke
 				(width 0.05)
@@
 		)
 		(fp_line
-			(start 1.3 1.3)
-			(end 1.3 -1.3)
+			(start 2.7 2.45)
+			(end 2.7 -2.45)
 			(stroke
 				(width 0.05)
@@
 		)
 		(fp_line
-			(start 2.3 -1.3)
-			(end 2.3 1.3)
+			(start 5.1 -2.45)
+			(end 5.1 2.45)
 			(stroke
 				(width 0.05)
@@
 		)
 		(fp_line
-			(start 2.3 1.3)
-			(end 4.9 1.3)
+			(start 5.1 2.45)
+			(end 10.5 2.45)
 			(stroke
 				(width 0.05)
@@
 		)
 		(fp_line
-			(start 4.9 -1.3)
-			(end 2.3 -1.3)
+			(start 10.5 -2.45)
+			(end 5.1 -2.45)
 			(stroke
 				(width 0.05)
@@
 		)
 		(fp_line
-			(start 4.9 1.3)
-			(end 4.9 -1.3)
+			(start 10.5 2.45)
+			(end 10.5 -2.45)
 			(stroke
 				(width 0.05)
@@
 		(fp_circle
 			(center 0 0)
-			(end 0.5 0)
+			(end 1.95 0)
 			(stroke
 				(width 0.1)
@@
 		)
 		(fp_circle
-			(center 3.6 0)
-			(end 4.1 0)
+			(center 7.8 0)
+			(end 9.75 0)
 			(stroke
 				(width 0.1)
@@
 		)
 		(fp_text user "${REFERENCE}"
-			(at 1.8 0 90)
+			(at 3.9 0 90)
 			(layer "F.Fab")
 			(effects
 				(font
-					(size 0.65 0.65)
-					(thickness 0.1)
+					(size 1 1)
+					(thickness 0.15)
 				)
 			)
@@
 		(pad "1" thru_hole roundrect
 			(at 0 0)
-			(size 1.6 1.6)
-			(drill 0.6)
+			(size 3.9 3.9)
+			(drill 2.5)
 			(layers "*.Cu" "*.Mask")
 			(remove_unused_layers no)
-			(roundrect_rratio 0.15625)
+			(roundrect_rratio 0.064103)
+			(net 7 "GND")
 		)
 		(pad "2" thru_hole circle
-			(at 3.6 0)
-			(size 1.6 1.6)
-			(drill 0.6)
+			(at 7.8 0)
+			(size 3.9 3.9)
+			(drill 2.5)
 			(layers "*.Cu" "*.Mask")
 			(remove_unused_layers no)
+			(net 2 "Net-(C1-Pad1)")
 		)
 		(embedded_fonts no)
-		(model "${KICAD9_3DMODEL_DIR}/Connector_Wire.3dshapes/SolderWire-0.1sqmm_1x02_P3.6mm_D0.4mm_OD1mm.wrl"
+		(model "${KICAD9_3DMODEL_DIR}/Connector_Wire.3dshapes/SolderWire-2sqmm_1x02_P7.8mm_D2mm_OD3.9mm.wrl"
 			(offset
 				(xyz 0 0 0)
@@
 	(footprint "Resistor_SMD:R_0805_2012Metric"
 		(layer "F.Cu")
-		(at 49 36.0375 -90)
+		(at 55.5 36.0375 -90)
 		(descr "Resistor SMD 0805 (2012 Metric), square (rectangular) end terminal, IPC_7351 nominal, (Body size source: IPC-SM-782 page 72, https://www.pcb-3d.com/wordpress/wp-content/uploads/ipc-sm-782a_amendment_1_and_2.pdf), generated with kicad-footprint-generator")
 		(tags "resistor")
@@
 		(at 49 44 -90)
 		(property "Reference" "U1"
-			(at -4.5 2 180)
+			(at -4.5 2 0)
 			(layer "F.SilkS")
 			(effects
@@
 		)
 		(embedded_fonts no)
+		(model "/Users/annagavrileva/Desktop/NE5532DR.STEP"
+			(offset
+				(xyz 0 0 0)
+			)
+			(scale
+				(xyz 1 1 1)
+			)
+			(rotate
+				(xyz -90 -0 -0)
+			)
+		)
 	)
 	(footprint "Connector_PinHeader_2.54mm:PinHeader_1x03_P2.54mm_Vertical"
@@
 		(layer "Edge.Cuts")
 	)
-	(gr_text "Team 50 - Design 1"
-		(at 58 35 0)
+	(gr_text "Team 50\nDesign 1"
+		(at 67.5 36 0)
 		(layer "F.SilkS" knockout)
 		(effects
@@
 	)
 	(segment
-		(start 51.375 35.125)
-		(end 51.5 35)
+		(start 57.875 35.125)
+		(end 58 35)
 		(width 0.2)
 		(layer "F.Cu")
@@
 	)
 	(segment
-		(start 49 35.125)
-		(end 51.375 35.125)
+		(start 55.5 35.125)
+		(end 57.875 35.125)
 		(width 0.2)
 		(layer "F.Cu")
@@
 	)
 	(segment
-		(start 51.5 36.9)
-		(end 53.9625 36.9)
+		(start 51 35.5)
+		(end 51.5 36)
+		(width 0.2)
+		(layer "F.Cu")
+		(net 2)
+	)
+	(segment
+		(start 60.1375 36.8625)
+		(end 60.1 36.9)
+		(width 0.2)
+		(layer "F.Cu")
+		(net 2)
+	)
+	(segment
+		(start 60.5 36.8625)
+		(end 60.1375 36.8625)
 		(width 0.2)
 		(layer "F.Cu")
@@
 	)
 	(segment
-		(start 53.9625 36.9)
-		(end 54 36.8625)
+		(start 60.4625 36.9)
+		(end 60.5 36.8625)
+		(width 0.2)
+		(layer "F.Cu")
+		(net 2)
+	)
+	(segment
+		(start 60.1 36.9)
+		(end 58 36.9)
+		(width 0.2)
+		(layer "F.Cu")
+		(net 2)
+	)
+	(segment
+		(start 57.1 36)
+		(end 58 36.9)
+		(width 0.2)
+		(layer "F.Cu")
+		(net 2)
+	)
+	(segment
+		(start 51.5 36)
+		(end 57.1 36)
 		(width 0.2)
 		(layer "F.Cu")
@@
 	)
 	(via
-		(at 37 39.5)
-		(size 0.6)
-		(drill 0.3)
-		(layers "F.Cu" "B.Cu")
-		(net 7)
-	)
-	(via
-		(at 72.5 43.5)
-		(size 0.6)
-		(drill 0.3)
-		(layers "F.Cu" "B.Cu")
-		(net 7)
-	)
-	(via
 		(at 59.9125 39)
 		(size 0.6)
@@
 	)
 	(segment
+		(start 54.699 37.751)
+		(end 55.5 36.95)
+		(width 0.2)
+		(layer "F.Cu")
+		(net 13)
+	)
+	(segment
 		(start 49 40.895)
 		(end 49.635 41.53)
@@
 	)
 	(segment
-		(start 49 36.95)
-		(end 49 39)
+		(start 49 39)
+		(end 50.249 37.751)
+		(width 0.2)
+		(layer "F.Cu")
+		(net 13)
+	)
+	(segment
+		(start 50.249 37.751)
+		(end 54.699 37.751)
 		(width 0.2)
 		(layer "F.Cu")
