File: Praxis_BeeFreq/Praxis_BeeFreq.kicad_sch (KiCad schematic)
At the start: 26 parts, among them J1 Conn_01x03_Pin, J2 UJC-HP-G-5-SMT-TR, U1 NE5532DR, U2 NE5532DR

Commit message: BetterVersion
Parts:
- removed J2: UJC-HP-G-5-SMT-TR, UJC-HP-G-5-SMT-TR:CUI_UJC-HP-G-5-SMT-TR, symbol UJC-HP-G-5-SMT-TR:UJC-HP-G-5-SMT-TR
- removed R5, R6: 5.1k, Resistor_SMD:R_0805_2012Metric, symbol Device:R
- C4: value 10n -> 11n
- MK2: footprint Connector_Wire:SolderWire-0.1sqmm_1x02_P3.6mm_D0.4mm_OD1mm -> Connector_Wire:SolderWire-2sqmm_1x02_P7.8mm_D2mm_OD3.9mm
Connections:
- no-connect marks 4 -> 3
Other:
- moved on the sheet: J1
